File: Modules/IO/Temp/pt1000/pt1000.kicad_sch (KiCad schematic)
At the start: 6 parts, among them U1 LM358

Commit message: 1
Parts:
- R1, R2, R3, R4: footprint (none) -> Resistor_SMD:R_0805_2012Metric
Changed lines of the file:
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@@
 			)
 		)
-		(property "Footprint" ""
+		(property "Footprint" "Resistor_SMD:R_0805_2012Metric"
 			(at 163.83 94.488 90)
 			(effects
@@
 			)
 		)
-		(property "Footprint" ""
+		(property "Footprint" "Resistor_SMD:R_0805_2012Metric"
 			(at 137.922 96.52 90)
 			(effects
@@
 			)
 		)
-		(property "Datasheet" "~"
+		(property "Datasheet" ""
 			(at 139.7 96.52 0)
 			(effects
@@
 			)
 		)
-		(property "Footprint" ""
+		(property "Footprint" "Resistor_SMD:R_0805_2012Metric"
 			(at 121.412 76.2 90)
 			(effects
@@
 			)
 		)
-		(property "Footprint" ""
+		(property "Footprint" "Resistor_SMD:R_0805_2012Metric"
 			(at 137.922 88.9 90)
 			(effects

Commit message: 1
Parts:
- removed TH1: PT1000, symbol Device:Thermistor
- added C1: 100nF, Capacitor_SMD:C_0805_2012Metric, symbol Device:C
- added J1, J2: Conn_01x02, Connector_Phoenix_MC:PhoenixContact_MCV_1,5_2-G-3.81_1x02_P3.81mm_Vertical, symbol Connector_Generic:Conn_01x02
- added R5, R6, R8: 10K, Resistor_SMD:R_0805_2012Metric, symbol Device:R
- added R7: 1K, Resistor_SMD:R_0805_2012Metric, symbol Device:R
- added unit 2 of U1
- added unit 3 of U1
- U1: footprint Package_DFN_QFN:DFN-8-1EP_2x2mm_P0.5mm_EP1.05x1.75mm -> Package_SO:SOIC-8-1EP_3.9x4.9mm_P1.27mm_EP2.29x3mm
Connections:
- net +5V: now also C1.2, R5.1, R6.1, U1.8 (V+)
- net GND: now also C1.1, J1.1 (Pin_1), J2.1 (Pin_1), R7.2, U1.4 (V-)
- net out1: now reaches R3.2, U1.1
- net at R2.2, U1.3 (+): now also J1.2 (Pin_2)
- new net: R6.2, R7.1, R8.1, U1.6 (-)
- new net: J2.2 (Pin_2), R5.2, U1.5 (+)
- new net out2: R8.2, U1.7
